File: V1/V1C06/exV1C06S02/exV1C06S02.kicad_sch (KiCad schematic)
At the start: 6 parts

Commit message: update V1 C05 C06 C07
Parts:
- removed BT1: 35, symbol Device:Battery_Cell
- removed BT2: 25, symbol Device:Battery_Cell
- added V1: 35, symbol Simulation_SPICE:VDC
- added V2: 25, symbol Simulation_SPICE:VDC
Connections:
- net 1: now also V1.1
- net 5: now also V2.2
- net GND: now also V1.2, V2.1
